Commit message: Add moveit packages and gazebo/moveit integration

File: warthog_arm/urdf/arm.xacro (robot description, xacro)
@@ -5,5 +5,5 @@
         <origin rpy="0 0 0" xyz="0 0 0"/>
         <geometry>
-          <mesh filename="package://manipulator_warthog/meshes/base.dae"/>
+          <mesh filename="package://warthog_arm/meshes/base.dae"/>
         </geometry>
       </visual>
@@ -11,10 +11,10 @@
         <origin rpy="0 0 0" xyz="0 0 0"/>
         <geometry>
-          <mesh filename="package://manipulator_warthog/meshes/base.dae"/>
+          <mesh filename="package://warthog_arm/meshes/base.dae"/>
         </geometry>
       </collision>
       <inertial>
         <origin rpy="0 0 0" xyz="0 0 0"/>
-        <mass value="10000.86661792"/>
+        <mass value="1.8"/>
         <inertia ixx="8.72078676" ixy="-9.55785583e-7" ixz="0" iyx="-9.55785583e-7" iyy="4.66430350" iyz="0" izx="0" izy="-0" izz="5.35109282"/>
       </inertial>
@@ -24,11 +24,11 @@
         <origin xyz="0 0 0" rpy="0 0 0" />
         <geometry>
-          <mesh filename="package://manipulator_warthog/meshes/id_1.dae"/>
-        </geometry>
-      </visual>
-      <collision>
-        <origin xyz="0 0 0" rpy="0 0 0" />
-        <geometry>
-          <mesh filename="package://manipulator_warthog/meshes/id_1.dae"/>
+          <mesh filename="package://warthog_arm/meshes/id_1.dae"/>
+        </geometry>
+      </visual>
+      <collision>
+        <origin xyz="0 0 0" rpy="0 0 0" />
+        <geometry>
+          <mesh filename="package://warthog_arm/meshes/id_1.dae"/>
         </geometry>
       </collision>
@@ -48,11 +48,11 @@
         <origin xyz="0 0 0" rpy="0 0 0" />
         <geometry>
-          <mesh filename="package://manipulator_warthog/meshes/id_2.dae"/>
-        </geometry>
-      </visual>
-      <collision>
-        <origin xyz="0 0 0" rpy="0 0 0" />
-        <geometry>
-          <mesh filename="package://manipulator_warthog/meshes/id_2.dae"/>
+          <mesh filename="package://warthog_arm/meshes/id_2.dae"/>
+        </geometry>
+      </visual>
+      <collision>
+        <origin xyz="0 0 0" rpy="0 0 0" />
+        <geometry>
+          <mesh filename="package://warthog_arm/meshes/id_2.dae"/>
         </geometry>
       </collision>
@@ -74,11 +74,11 @@
         <origin xyz="0 0 0" rpy="0 0 0" />
         <geometry>
-          <mesh filename="package://manipulator_warthog/meshes/id_3.dae"/>
-        </geometry>
-      </visual>
-      <collision>
-        <origin xyz="0 0 0" rpy="0 0 0" />
-        <geometry>
-          <mesh filename="package://manipulator_warthog/meshes/id_3.dae"/>
+          <mesh filename="package://warthog_arm/meshes/id_3.dae"/>
+        </geometry>
+      </visual>
+      <collision>
+        <origin xyz="0 0 0" rpy="0 0 0" />
+        <geometry>
+          <mesh filename="package://warthog_arm/meshes/id_3.dae"/>
         </geometry>
       </collision>
@@ -100,11 +100,11 @@
         <origin xyz="0 0 0" rpy="0 0 0" />
         <geometry>
-          <mesh filename="package://manipulator_warthog/meshes/id_4.dae"/>
-        </geometry>
-      </visual>
-      <collision>
-        <origin xyz="0 0 0" rpy="0 0 0" />
-        <geometry>
-          <mesh filename="package://manipulator_warthog/meshes/id_4.dae"/>
+          <mesh filename="package://warthog_arm/meshes/id_4.dae"/>
+        </geometry>
+      </visual>
+      <collision>
+        <origin xyz="0 0 0" rpy="0 0 0" />
+        <geometry>
+          <mesh filename="package://warthog_arm/meshes/id_4.dae"/>
         </geometry>
       </collision>
@@ -126,11 +126,11 @@
         <origin xyz="0 0 0" rpy="0 0 0" />
         <geometry>
-          <mesh filename="package://manipulator_warthog/meshes/id_5.dae"/>
-        </geometry>
-      </visual>
-      <collision>
-        <origin xyz="0 0 0" rpy="0 0 0" />
-        <geometry>
-          <mesh filename="package://manipulator_warthog/meshes/id_5.dae"/>
+          <mesh filename="package://warthog_arm/meshes/id_5.dae"/>
+        </geometry>
+      </visual>
+      <collision>
+        <origin xyz="0 0 0" rpy="0 0 0" />
+        <geometry>
+          <mesh filename="package://warthog_arm/meshes/id_5.dae"/>
         </geometry>
       </collision>
@@ -153,5 +153,5 @@
         <origin xyz="0.0 0.0 0.0" rpy="0 0 0" />
         <geometry>
-          <mesh filename="package://manipulator_warthog/meshes/id_6.dae"/>
+          <mesh filename="package://warthog_arm/meshes/id_6.dae"/>
         </geometry>
       </visual>
@@ -159,5 +159,5 @@
         <origin xyz="0.0 0.0 0.0" rpy="0 0 0" />
         <geometry>
-          <mesh filename="package://manipulator_warthog/meshes/id_6.dae"/>
+          <mesh filename="package://warthog_arm/meshes/id_6.dae"/>
         </geometry>
       </collision>
